Commit message: Imported upstream version '0.7.3' of 'upstream'

File: heifu_description/models/heifu_with_ardupilot/model.sdf.xacro (robot description, xacro)
@@ -25,4 +25,78 @@
           </axis>
         </joint>-->
+      <!-- CameraLink -->
+      <xacro:macro name="camera_plugin_xacro" params="name">
+        <link name="camera_link">
+          <pose>0.3 0 0.4 0 0 0</pose>
+            <inertial>
+              <pose>0 0 0 0 -0 0</pose>
+              <mass>0.01</mass>
+              <inertia>
+                <ixx>4.15e-6</ixx>
+                <ixy>0</ixy>
+                <ixz>0</ixz>
+                <iyy>2.407e-6</iyy>
+                <iyz>0</iyz>
+                <izz>2.407e-6</izz>
+              </inertia>
+            </inertial>
+            <visual name="visual">
+              <geometry>
+                <box>
+                  <size>0.005 0.005 0.005</size>
+                </box>
+              </geometry>
+              <material>
+                <script>
+                  <name>Gazebo/DarkGrey</name>
+                </script>
+              </material>
+            </visual>
+            <!-- camera -->
+            <sensor type="depth" name="pointcloud_sensor">
+                <always_on>1</always_on>
+                <visualize>true</visualize>
+                <camera>
+                  <horizontal_fov>1.047</horizontal_fov>
+                  <image>
+                      <width>640</width>
+                      <height>480</height>
+                      <format>R8G8B8</format>
+                  </image>
+                  <depth_camera>
+                  </depth_camera>
+                  <clip>
+                      <near>0.1</near>
+                      <far>100</far>
+                  </clip>
+                </camera>
+                <plugin name="camera_controller" filename="libgazebo_ros_openni_kinect.so">
+                  <robotNamespace>${name}</robotNamespace>
+                  <alwaysOn>true</alwaysOn>
+                  <updateRate>10.0</updateRate>
+                  <cameraName>pointcloud</cameraName>
+                  <frameName>camera_link</frameName>
+                  <imageTopicName>color/image_raw</imageTopicName>
+                  <depthImageTopicName>depth/image_raw</depthImageTopicName>
+                  <pointCloudTopicName>depth/color/points</pointCloudTopicName>
+                  <cameraInfoTopicName>color/camera_info</cameraInfoTopicName>
+                  <depthImageCameraInfoTopicName>depth/camera_info</depthImageCameraInfoTopicName>
+                  <pointCloudCutoffMax>10.0</pointCloudCutoffMax>
+                  <pointCloudCutoff>1.0</pointCloudCutoff>
+                  <hackBaseline>0.07</hackBaseline>
+                  <distortionK1>0.0</distortionK1>
+                  <distortionK2>0.0</distortionK2>
+                  <distortionK3>0.0</distortionK3>
+                  <distortionT1>0.0</distortionT1>
+                  <distortionT2>0.0</distortionT2>
+                  <CxPrime>0.0</CxPrime>
+                  <Cx>0.0</Cx>
+                  <Cy>0.0</Cy>
+                  <focalLength>0.0</focalLength>
+                </plugin>
+              </sensor>
+          </link>
+        </xacro:macro>
+        <xacro:camera_plugin_xacro name="$(arg name)"/>
         <!-- plugins -->
         <xacro:macro name="rotor_plugin_macro" params="motor_number blade_number fw_force cp">

Commit message: Rebase from 'upstream'

File: heifu_description/models/heifu_with_ardupilot/model.sdf.xacro (robot description, xacro)
@@ -25,78 +25,4 @@
           </axis>
         </joint>-->
-      <!-- CameraLink -->
-      <xacro:macro name="camera_plugin_xacro" params="name">
-        <link name="camera_link">
-          <pose>0.3 0 0.4 0 0 0</pose>
-            <inertial>
-              <pose>0 0 0 0 -0 0</pose>
-              <mass>0.01</mass>
-              <inertia>
-                <ixx>4.15e-6</ixx>
-                <ixy>0</ixy>
-                <ixz>0</ixz>
-                <iyy>2.407e-6</iyy>
-                <iyz>0</iyz>
-                <izz>2.407e-6</izz>
-              </inertia>
-            </inertial>
-            <visual name="visual">
-              <geometry>
-                <box>
-                  <size>0.005 0.005 0.005</size>
-                </box>
-              </geometry>
-              <material>
-                <script>
-                  <name>Gazebo/DarkGrey</name>
-                </script>
-              </material>
-            </visual>
-            <!-- camera -->
-            <sensor type="depth" name="pointcloud_sensor">
-                <always_on>1</always_on>
-                <visualize>true</visualize>
-                <camera>
-                  <horizontal_fov>1.047</horizontal_fov>
-                  <image>
-                      <width>640</width>
-                      <height>480</height>
-                      <format>R8G8B8</format>
-                  </image>
-                  <depth_camera>
-                  </depth_camera>
-                  <clip>
-                      <near>0.1</near>
-                      <far>100</far>
-                  </clip>
-                </camera>
-                <plugin name="camera_controller" filename="libgazebo_ros_openni_kinect.so">
-                  <robotNamespace>${name}</robotNamespace>
-                  <alwaysOn>true</alwaysOn>
-                  <updateRate>10.0</updateRate>
-                  <cameraName>pointcloud</cameraName>
-                  <frameName>camera_link</frameName>
-                  <imageTopicName>color/image_raw</imageTopicName>
-                  <depthImageTopicName>depth/image_raw</depthImageTopicName>
-                  <pointCloudTopicName>depth/color/points</pointCloudTopicName>
-                  <cameraInfoTopicName>color/camera_info</cameraInfoTopicName>
-                  <depthImageCameraInfoTopicName>depth/camera_info</depthImageCameraInfoTopicName>
-                  <pointCloudCutoffMax>10.0</pointCloudCutoffMax>
-                  <pointCloudCutoff>1.0</pointCloudCutoff>
-                  <hackBaseline>0.07</hackBaseline>
-                  <distortionK1>0.0</distortionK1>
-                  <distortionK2>0.0</distortionK2>
-                  <distortionK3>0.0</distortionK3>
-                  <distortionT1>0.0</distortionT1>
-                  <distortionT2>0.0</distortionT2>
-                  <CxPrime>0.0</CxPrime>
-                  <Cx>0.0</Cx>
-                  <Cy>0.0</Cy>
-                  <focalLength>0.0</focalLength>
-                </plugin>
-              </sensor>
-          </link>
-        </xacro:macro>
-        <xacro:camera_plugin_xacro name="$(arg name)"/>
         <!-- plugins -->
         <xacro:macro name="rotor_plugin_macro" params="motor_number blade_number fw_force cp">
